Commit message: Update turtlebot3_waffle_pi.urdf.xacro

File: turtlebot3_waffle_pi.urdf.xacro (robot description, xacro)
@@ -3,8 +3,6 @@
   <xacro:include filename="$(find turtlebot3_description)/urdf/common_properties.xacro"/>
   <xacro:include filename="$(find turtlebot3_description)/urdf/turtlebot3_waffle_pi.gazebo.xacro"/>
-  <!-- <xacro:include filename="$(find realsense2_description)/urdf/_d435.urdf.xacro" /> -->
   <xacro:include filename="$(find turtlebot3_description)/urdf/_d435i.urdf.xacro" />
   <xacro:sensor_d435i parent="base_link" name="D435i_camera" topics_ns="D435i_camera">
-  <!-- <xacro:sensor_d435i name="camera" topics_ns="camera" parent="base_link" publish_pointcloud="true"> -->
     <origin xyz="0.049 0.0 0.055" rpy="0 0 0" />
   </xacro:sensor_d435i>
@@ -166,28 +164,3 @@
     </inertial>
   </link>
-  <!-- <joint name="camera_joint" type="fixed">
-    <origin xyz="0.073 -0.011 0.084" rpy="0 0 0"/>
-    <parent link="base_link"/>
-    <child link="camera_link"/>
-  </joint>
-  <link name="camera_link">
-    <collision>
-      <origin xyz="0.005 0.011 0.013" rpy="0 0 0"/>
-      <geometry>
-        <box size="0.015 0.030 0.027"/>
-      </geometry>
-    </collision>
-  </link>
-  <joint name="camera_rgb_joint" type="fixed">
-    <origin xyz="0.003 0.011 0.009" rpy="0 0 0"/>
-    <parent link="camera_link"/>
-    <child link="camera_rgb_frame"/>
-  </joint>
-  <link name="camera_rgb_frame"/>
-  <joint name="camera_rgb_optical_joint" type="fixed">
-    <origin xyz="0 0 0" rpy="-1.57 0 -1.57"/>
-    <parent link="camera_rgb_frame"/>
-    <child link="camera_rgb_optical_frame"/>
-  </joint>
-  <link name="camera_rgb_optical_frame"/> -->
 </robot>
